File: electronics/rodl/rodl.kicad_pcb (KiCad board)
At the start: 2 copper layers, 16 parts, among them Q1 AO4805_C5183840, U1 ESP32-S3-MINI-1U-N8, U2 TPS54302DDCR_C311983, U3 HUSB237-AA001-DN06R, U4 DOS4427

Commit message: new electronic version
Parts:
- removed USB1: TYPE-C 16PIN 2MD(073), rodl:USB-C-SMD_TYPE-C-6PIN-2MD-073
- added C10: 100nF, Capacitor_SMD:C_0603_1608Metric, F.Cu at (229.8, 85.2)
- added C11: 10uF, Capacitor_SMD:C_0603_1608Metric, F.Cu at (229.8, 87.7)
- added C12: 100nF, Capacitor_SMD:C_0603_1608Metric, F.Cu at (233.8, 77.7)
- added C13: 10uF, Capacitor_SMD:C_0603_1608Metric, F.Cu at (233.8, 80.2)
- added C14: 100nF, Capacitor_SMD:C_0603_1608Metric, F.Cu at (233.8, 82.7)
- added C15: 10uF, Capacitor_SMD:C_0603_1608Metric, F.Cu at (161.3, 95.1)
- added C16: 100nF, Capacitor_SMD:C_0603_1608Metric, F.Cu at (161.3, 97.6)
- added C7: 1uF, Capacitor_SMD:C_0603_1608Metric, F.Cu at (123.9, 76.7)
- added C8: 10uF, Capacitor_SMD:C_0603_1608Metric, F.Cu at (229.8, 80.2)
- added C9: 100nF, Capacitor_SMD:C_0603_1608Metric, F.Cu at (229.8, 82.7)
- added CN1: ATGM336H-6N-74, rodl:COMM-SMD_18P-L10.1-W9.7-P1.1-TL_L76-LB, F.Cu at (165.8, 88.3)
- added D1: LED, LED_SMD:LED_0603_1608Metric, F.Cu at (165.4, 105.2)
- added H1: MountingHole_Pad, MountingHole:MountingHole_2.5mm_Pad_TopOnly, F.Cu at (243.1, 79.7)
- added H2: MountingHole_Pad, MountingHole:MountingHole_2.5mm_Pad_TopOnly, F.Cu at (156.0, 85.8)
- added H3: MountingHole_Pad, MountingHole:MountingHole_2.5mm_Pad_TopOnly, F.Cu at (156.0, 92.3)
- added H4: MountingHole_Pad, MountingHole:MountingHole_2.5mm_Pad_TopOnly, F.Cu at (156.0, 98.9)
- added J1: ~, Connector_PinSocket_2.54mm:PinSocket_2x03_P2.54mm_Vertical, F.Cu at (129.7, 77.6)
- added J2: Conn_01x03_Pin, Connector_PinSocket_2.00mm:PinSocket_1x03_P2.00mm_Vertical, F.Cu at (176.6, 95.9)
- added J3: Conn_01x04_Pin, Connector_PinSocket_2.00mm:PinSocket_1x04_P2.00mm_Vertical, F.Cu at (165.3, 95.9)
- added J4: Conn_01x09, rodl:Connector_Rodl, F.Cu at (98.5, 77.6)
- added L2: 39nH, Inductor_SMD:L_0603_1608Metric, F.Cu at (161.3, 100.2)
- added Q2: AO3415_C840839, rodl:SOT-23-3_L2.9-W1.6-P1.90-LS2.8-BR, F.Cu at (242.1, 89.7)
- added R10: 220, Resistor_SMD:R_0603_1608Metric, F.Cu at (161.3, 102.7)
- added R11: NC, Resistor_SMD:R_0603_1608Metric, F.Cu at (161.3, 105.2)
- added R12: 220, Resistor_SMD:R_0603_1608Metric, F.Cu at (191.2, 106.2)
- added R13: 220, Resistor_SMD:R_0603_1608Metric, F.Cu at (191.2, 108.7)
- added R14: 220, Resistor_SMD:R_0603_1608Metric, F.Cu at (191.2, 111.2)
- added R4: 10k, Resistor_SMD:R_0603_1608Metric, F.Cu at (123.9, 79.7)
- added R5: NC, Resistor_SMD:R_0603_1608Metric, F.Cu at (233.8, 87.7)
- added R6: 10k, Resistor_SMD:R_0603_1608Metric, F.Cu at (237.8, 77.7)
- added R7: 10k, Resistor_SMD:R_0603_1608Metric, F.Cu at (237.8, 80.2)
- added R8: 10k, Resistor_SMD:R_0603_1608Metric, F.Cu at (237.8, 82.7)
- added R9: 1k, Resistor_SMD:R_0603_1608Metric, F.Cu at (237.8, 85.2)
- added U5: LIS3DHTR_C15134, rodl:LGA-16_L3.0-W3.0-P0.50-TL, F.Cu at (242.5, 85.3)
- added U6: BWU.FL-IPEX1, rodl:IPEX-SMD_BWIPX-1-001E, F.Cu at (154.6, 104.6)
- added USB2: GT-USB-7055BB, rodl:USB-C-TH_GT-USB-7055BB, F.Cu at (232.9, 92.2)
- moved C1 59.8 mm to (202.1, 80.3)
- moved C2 59.8 mm to (202.1, 82.8)
- moved C3 59.8 mm to (202.1, 85.3)
- moved C4 59.8 mm to (219.8, 89.6)
- moved C5 59.8 mm to (219.8, 92.6)
- moved C6 59.8 mm to (202.1, 87.8)
- moved L1 59.8 mm to (214.0, 91.7)
- moved Q1 59.8 mm to (207.2, 92.2)
- moved R1 59.8 mm to (202.1, 90.3)
- moved R2 59.8 mm to (202.1, 92.8)
- moved R3 59.8 mm to (202.1, 95.4)
- moved U2 59.8 mm to (212.8, 97.5)
- moved U3 59.8 mm to (219.8, 95.8)
- moved U4 59.8 mm to (218.8, 83.2)
- moved U1 17.1 mm to (115.2, 83.5)
Connections:
- Q1 pad 1: unconnected-(Q1-S2-Pad1) -> USB_VIN
- Q1 pad 2: unconnected-(Q1-G2-Pad2) -> /DOS_OUTA
- Q1 pad 3: unconnected-(Q1-S1-Pad3) -> USB_VIN
- Q1 pad 4: unconnected-(Q1-G1-Pad4) -> /DOS_OUTB
- Q1 pad 5: unconnected-(Q1-D1-Pad5) -> /LED_LOW
- Q1 pad 6: unconnected-(Q1-D1-Pad6) -> /LED_LOW
- Q1 pad 7: unconnected-(Q1-D2-Pad7) -> /LED_HIGH
- Q1 pad 8: unconnected-(Q1-D2-Pad8) -> /LED_HIGH
- U1 pad 21: unconnected-(U1-IO17-Pad21) -> /GPS_RX
- U1 pad 22: unconnected-(U1-IO18-Pad22) -> /GPS_TX
- U1 pad 23: unconnected-(U1-IO19-Pad23) -> /USB_D-
- U1 pad 24: unconnected-(U1-IO20-Pad24) -> /USB_D+
- U1 pad 3: unconnected-(U1-3V3-Pad3) -> +3.3V
- U1 pad 39: unconnected-(U1-TXD0-Pad39) -> /ESP_TX
- U1 pad 4: unconnected-(U1-IO0-Pad4) -> /ESP_IO0
- U1 pad 40: unconnected-(U1-RXD0-Pad40) -> /ESP_RX
- U1 pad 45: unconnected-(U1-EN-Pad45) -> /ESP_EN
- U1 pad 8: unconnected-(U1-IO4-Pad8) -> /LED_HIGH_C
- U1 pad 9: unconnected-(U1-IO5-Pad9) -> /LED_LOW_C
- U3 pad 1: unconnected-(U3-CC1-Pad1) -> /USB_CC1
- U3 pad 2: unconnected-(U3-VUSB-Pad2) -> USB_VIN
- U3 pad 3: unconnected-(U3-VSET-Pad3) -> Net-(U3-VSET)
- U3 pad 6: unconnected-(U3-CC2-Pad6) -> /USB_CC2
- U3 pad 7: unconnected-(U3-GND-Pad7) -> GND
- U4 pad 2: unconnected-(U4-INA-Pad2) -> /LED_HIGH_C
- U4 pad 3: unconnected-(U4-GND-Pad3) -> GND
- U4 pad 4: unconnected-(U4-INB-Pad4) -> /LED_LOW_C
- U4 pad 5: unconnected-(U4-OUTB-Pad5) -> /DOS_OUTB
- U4 pad 6: unconnected-(U4-VCC-Pad6) -> USB_VIN
- U4 pad 7: unconnected-(U4-OUTA-Pad7) -> /DOS_OUTA
Other:
- board outline added: 49.2 x 29.9 mm
- copper layers 2 -> 6

Commit message: finish pcb
Parts:
- removed H3: MountingHole_Pad, MountingHole:MountingHole_2.5mm_Pad_TopOnly
- added C17: 10uF, Capacitor_SMD:C_0603_1608Metric, F.Cu at (104.7, 100.5)
- added C18: 10uF, Capacitor_SMD:C_0603_1608Metric, F.Cu at (101.9, 96.7)
- added C19: 100nF, Capacitor_SMD:C_0603_1608Metric, F.Cu at (104.7, 102.0)
- added G***: LOGO, logo:qr, B.Cu at (115.2, 83.2)
- added G***: LOGO, logo:logo, B.Cu at (95.7, 91.7)
- added U7: HT7550-1_C41355185, rodl:SOT-89-3_L4.5-W2.4-P1.50-LS4.0-BR, F.Cu at (105.3, 97.2)
- added U8: SN74AHCT1G125DCKR, rodl:SC-70-5_L2.0-W1.3-P0.65-LS2.1-BL, F.Cu at (101.6, 101.2)
- C15, C16, CN1, D1, L2, R10: moved to B.Cu
- moved Q2 144.9 mm to (97.3, 82.3), turned to -90 degrees
- moved R5 144.9 mm to (88.9, 84.4)
- moved USB2 144.5 mm to (89.0, 78.3)
- moved R8 143.0 mm to (94.8, 82.3), turned to 90 degrees
- moved R9 140.4 mm to (97.4, 85.2), turned to 180 degrees
- moved U5 139.3 mm to (103.2, 90.3)
- moved R7 138.1 mm to (100.0, 90.1), turned to -90 degrees
- moved R6 135.5 mm to (103.2, 93.2), turned to 180 degrees
- moved U3 131.6 mm to (88.9, 82.4)
- moved C12 129.6 mm to (104.5, 87.1)
- moved C10 128.4 mm to (101.4, 87.1), turned to 180 degrees
- moved C5 126.8 mm to (93.1, 97.6)
- moved C11 125.3 mm to (104.5, 85.6)
- moved C8 125.1 mm to (104.7, 78.4), turned to 90 degrees
- moved C9 123.6 mm to (106.2, 78.4), turned to 90 degrees
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Connections:
- C1 pad 1: +12V -> USB_VIN
- C2 pad 1: +12V -> USB_VIN
- U1 pad 10: unconnected-(U1-IO6-Pad10) -> /+3.3V_T
- U1 pad 13: unconnected-(U1-IO9-Pad13) -> /ACC_SCL
- U1 pad 14: unconnected-(U1-IO10-Pad14) -> /ACC_SDA
- U1 pad 15: unconnected-(U1-IO11-Pad15) -> /ACC_INT
- U1 pad 16: unconnected-(U1-IO12-Pad16) -> /WS_D_3.3
- U1 pad 17: unconnected-(U1-IO13-Pad17) -> /LED_LOW_C
- U1 pad 18: unconnected-(U1-IO14-Pad18) -> /LED_HIGH_C
- U1 pad 42: unconnected-(U1-GND-Pad42) -> GND
- U1 pad 43: unconnected-(U1-GND-Pad43) -> GND
- U1 pad 5: unconnected-(U1-IO1-Pad5) -> /LED_GPS
- U1 pad 6: unconnected-(U1-IO2-Pad6) -> /LED_BTN
- U1 pad 8: /LED_HIGH_C -> /BTN
- U1 pad 9: /LED_LOW_C -> /POTI
- U2 pad 3: +12V -> USB_VIN
Routing:
- net /USB_D-: track 0.00 -> 39.8 mm, vias 0 -> 2
- net /USB_D+: track 0.00 -> 39.0 mm, vias 0 -> 3
- net /ESP_IO0: track 0.00 -> 22.5 mm, vias 0 -> 1
- net USB_VIN: track 0.00 -> 15.8 mm, vias 0 -> 28
- net Net-(J4-Pin_9): track 0.00 -> 13.5 mm, vias 0 -> 1
- net /WS_D_3.3: track 0.00 -> 12.9 mm, vias 0 -> 2
- net /ESP_EN: track 0.00 -> 12.8 mm, vias 0 -> 1
- net /GPS_TX: track 0.00 -> 12.6 mm, vias 0 -> 2
- net /POTI: track 0.00 -> 11.6 mm, vias 0 -> 1
- net /ACC_SCL: track 0.00 -> 11.4 mm, vias 0 -> 2
- net /GPS_RX: track 0.00 -> 11.3 mm, vias 0 -> 2
- net /LED_HIGH: track 0.00 -> 10.3 mm
- net /+3.3V_T: track 0.00 -> 10.2 mm, vias 0 -> 2
- net /ACC_SDA: track 0.00 -> 9.87 mm, vias 0 -> 2
- net /USB_CC1: track 0.00 -> 8.27 mm, vias 0 -> 2
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- added copper zone on B.Cu, net +3.3V
- added copper zone on F.Cu, net +3.3V
- added copper zone on In2.Cu, net +3.3V
- added copper zone on F.Cu, net +5V
- added copper zone on F.Cu, net /DOS_OUTA
- added copper zone on F.Cu, net /DOS_OUTB
- added copper zone on F.Cu, net /FB_TPS
- added copper zone on F.Cu, net /LED_HIGH
- added copper zone on F.Cu, net /LED_LOW
- added copper zone on F.Cu, net /SW_TPS
- added copper zone on B.Cu, net GND
- added copper zone on F.Cu, net GND
- added copper zone on In1.Cu, net GND
- added copper zone on In4.Cu, net GND
- added copper zone on F.Cu, net Net-(C6-Pad1)
- added copper zone on B.Cu, net Net-(D1-A)
- added copper zone on F.Cu, net Net-(Q2-G)
- added copper zone on F.Cu, net Net-(U2-BOOT)
- added copper zone on F.Cu, net Net-(U3-VSET)
- added copper zone on F.Cu, net USB_VIN
- added copper zone on In2.Cu, net USB_VIN
Other:
- board text added: "3.3"
- board text added: "3.3V"
- board text added: "B"
- board text added: "BTN"
- board text added: "D"
- board text added: "EN"
- board text added: "G"
- board text added: "GND"
- board text added: "GPS"
- board text added: "GPS ANT"
- board text added: "H"
- board text added: "IO0"
- board text added: "L"
- board text added: "LED"
- board text added: "POT"
- board text added: "RX"
- board text added: "TX"
- board text added: "V"
- board text added: "WS2815"
