File: electronics/rodl/rodl.kicad_sch (KiCad schematic)
At the start: 27 parts, among them Q1 AO4805_C5183840, U1 ESP32-S3-MINI-1U-N8, U2 TPS54302DDCR_C311983, U3 HUSB237-AA001-DN06R, U4 DOS4427, U5 LIS3DHTR_C15134

Commit message: new electronic version
Parts:
- removed USB1: TYPE-C 16PIN 2MD(073), rodl:USB-C-SMD_TYPE-C-6PIN-2MD-073, symbol rodl:TYPE-C16PIN2MD(073)
- added C13, C15: 10uF, Capacitor_SMD:C_0603_1608Metric, symbol Device:C
- added C14, C16: 100nF, Capacitor_SMD:C_0603_1608Metric, symbol Device:C
- added CN1: ATGM336H-6N-74, rodl:COMM-SMD_18P-L10.1-W9.7-P1.1-TL_L76-LB, symbol rodl:ATGM336H-6N-74
- added D1: LED, LED_SMD:LED_0603_1608Metric, symbol Device:LED
- added H1, H2, H3, H4: MountingHole_Pad, MountingHole:MountingHole_2.5mm_Pad_TopOnly, symbol Mechanical:MountingHole_Pad
- added J1: ~, Connector_PinSocket_2.54mm:PinSocket_2x03_P2.54mm_Vertical, symbol Connector_Generic:Conn_02x03_Counter_Clockwise
- added J2: Conn_01x03_Pin, Connector_PinSocket_2.00mm:PinSocket_1x03_P2.00mm_Vertical, symbol Connector:Conn_01x03_Pin
- added J3: Conn_01x04_Pin, Connector_PinSocket_2.00mm:PinSocket_1x04_P2.00mm_Vertical, symbol Connector:Conn_01x04_Pin
- added J4: Conn_01x09, rodl:Connector_Rodl, symbol Connector_Generic:Conn_01x09
- added L2: 39nH, Inductor_SMD:L_0603_1608Metric, symbol Device:L
- added Q2: AO3415_C840839, rodl:SOT-23-3_L2.9-W1.6-P1.90-LS2.8-BR, symbol rodl:AO3415_C840839
- added R10, R12, R13, R14: 220, Resistor_SMD:R_0603_1608Metric, symbol Device:R
- added R11: NC, Resistor_SMD:R_0603_1608Metric, symbol Device:R
- added R8: 10k, Resistor_SMD:R_0603_1608Metric, symbol Device:R
- added R9: 1k, Resistor_SMD:R_0603_1608Metric, symbol Device:R
- added U6: BWU.FL-IPEX1, rodl:IPEX-SMD_BWIPX-1-001E, symbol rodl:BWU.FL-IPEX1
- added USB2: GT-USB-7055BB, rodl:USB-C-TH_GT-USB-7055BB, symbol rodl:GT-USB-7055BB
Connections:
- net +3.3V: now also C15.1, C16.1, CN1.6 (VBAT), CN1.8 (VCC), Q2.2 (S), R11.2
- net ESP_EN: now also J1.3 (Pin_3)
- net GND: now also U4.3 (GND), C13.2, C14.2, C15.2, C16.2, CN1.1 (GND), CN1.10 (GND), CN1.12 (GND), D1.1 (K), H1.1, H2.1, H3.1, H4.1, J1.5 (Pin_5), J2.2 (Pin_2), J3.2 (Pin_2), J3.3 (Pin_3), J4.1 (Pin_1), J4.4 (Pin_4), J4.5 (Pin_5), J4.7 (Pin_7), U6.2, U6.3, USB2.17 (EH), USB2.A1 (GND), USB2.A12 (GND), USB2.B1 (GND), USB2.B12 (GND)
- net USB_CC1: now also USB2.A5 (CC1)
- net USB_CC2: now also USB2.B5 (CC2)
- net USB_D+: now also USB2.A6 (D+), USB2.B6 (D+)
- net USB_D-: now also USB2.A7 (D-), USB2.B7 (D-)
- net USB_VIN: now also Q1.1 (S2), Q1.3 (S1), U4.6 (VCC), C13.1, C14.1, J3.1 (Pin_1), USB2.A4 (VBUS), USB2.A9 (VBUS), USB2.B4 (VBUS), USB2.B9 (VBUS)
- net LED_HIGH_C: now reaches U4.2 (INA)
- net LED_HIGH_C: now also U1.8 (IO4)
- net LED_LOW_C: now reaches U4.4 (INB)
- net LED_LOW_C: now also U1.9 (IO5)
- net DOS_OUTB: now reaches U4.5 (OUTB)
- net DOS_OUTB: now also Q1.4 (G1)
- net DOS_OUTA: now reaches U4.7 (OUTA)
- net DOS_OUTA: now also Q1.2 (G2)
- net GPS_RX: now reaches U1.21 (IO17)
- net GPS_RX: now also CN1.3 (RXD0)
- net GPS_TX: now reaches U1.22 (IO18)
- net GPS_TX: now also CN1.2 (TXD0)
- net ESP_TX: now reaches U1.39 (TXD0)
- net ESP_TX: now also J1.2 (Pin_2)
- net ESP_RX: now reaches U1.40 (RXD0)
- net ESP_RX: now also J1.1 (Pin_1)
- net LED_LOW: now reaches Q1.5 (D1)
- net LED_LOW: now also Q1.6 (D1), J2.3 (Pin_3)
- net LED_HIGH: now reaches Q1.7 (D2)
- net LED_HIGH: now also Q1.8 (D2), J2.1 (Pin_1)
- net IO0 renamed ESP_IO0
- net ESP_IO0: now also J1.6 (Pin_6)
- new net: D1.2 (A), R10.1
- new net: J4.2 (Pin_2), R12.1
- new net: J4.3 (Pin_3), R13.1
- new net: J4.9 (Pin_9), R14.1
- new net: CN1.11 (RF_IN), L2.2, U6.1
- new net: CN1.14 (VCC_RF), L2.1
- new net: CN1.4 (1PPS), R10.2
- new net: J1.4 (Pin_4), R11.1
- new net: Q2.1 (G), R8.1, R9.2
- new net +3.3V_C: J4.8 (Pin_8), Q2.3 (D), R8.2
- new net +3.3V_T: R9.1
- new net BTN: R14.2
- new net LED_BTN: R13.2
- new net LED_GPS: R12.2
- new net POTI: J4.6 (Pin_6)
- new net WS_D: J3.4 (Pin_4)
Other:
- note added: "1-2: GPS Status LED 3: Button LED Control 4: Poti GND 5: Button LED GND 6: Poti Signal 7: Button GND 8: Poti VCC 9: Button"
- note added: "Debug LED"
- note added: "Headlight"
- note added: "LEDs"
- note added: "UART Debug"
- moved on the sheet: C1, C10, C11, C12, C2, C3, C4, C5, C6, C7, C8, C9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

Commit message: finish pcb
Parts:
- removed H3: MountingHole_Pad, MountingHole:MountingHole_2.5mm_Pad_TopOnly, symbol Mechanical:MountingHole_Pad
- added C17, C18: 10uF, Capacitor_SMD:C_0603_1608Metric, symbol Device:C
- added C19: 100nF, Capacitor_SMD:C_0603_1608Metric, symbol Device:C
- added U7: HT7550-1_C41355185, rodl:SOT-89-3_L4.5-W2.4-P1.50-LS4.0-BR, symbol rodl:HT7550-1_C41355185
- added U8: SN74AHCT1G125DCKR, rodl:SC-70-5_L2.0-W1.3-P0.65-LS2.1-BL, symbol rodl:SN74AHCT1G125DCKR
Connections:
- net +12V is gone; now on net USB_VIN: C1.1, C2.1, U2.3 (VIN)
- net +3.3V_T: now also U1.10 (IO6)
- net ACC_INT: now also U1.15 (IO11)
- net ACC_SCL: now also U1.13 (IO9)
- net ACC_SDA: now also U1.14 (IO10)
- net BTN: now also U1.8 (IO4)
- net GND: now also U1.42 (GND), U1.43 (GND), C17.2, C18.1, C19.2, U7.1 (GND), U8.3 (GND)
- net LED_BTN: now also U1.6 (IO2)
- net LED_GPS: now also U1.5 (IO1)
- net LED_HIGH_C: now also U1.18 (IO14); no longer U1.8 (IO4)
- net LED_LOW_C: now also U1.17 (IO13); no longer U1.9 (IO5)
- net POTI: now also U1.9 (IO5)
- net USB_VIN: now also C18.2, U7.2 (VIN)
- net WS_D: now also U8.4 (Y)
- net WS_D_3.3: now reaches U1.16 (IO12)
- net WS_D_3.3: now also U8.2 (A)
- new net +5V: C17.1, C19.1, U7.3 (VOUT), U8.5 (VCC)
Other:
- note added: "5V Supply for Level Shifter"
- note added: "Level Shifter for WS2815"

Commit message: change structure
Connections:
- net +3.3V: now also Q2.3 (D); no longer Q2.2 (S)
- net +3.3V_C: now also Q2.2 (S); no longer Q2.3 (D)
Other:
- moved on the sheet: Q2, R8, R9
Changed lines of the file:
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@@
 	)
 	(junction
-		(at 236.22 250.19)
-		(diameter 0)
-		(color 0 0 0 0)
-	)
-	(junction
 		(at 91.44 40.64)
 		(diameter 0)
@@
 	)
 	(junction
+		(at 250.19 260.35)
+		(diameter 0)
+		(color 0 0 0 0)
+	)
+	(junction
 		(at 215.9 175.26)
 		(diameter 0)
@@
 	)
 	(junction
+		(at 236.22 250.19)
+		(diameter 0)
+		(color 0 0 0 0)
+	)
+	(junction
 		(at 160.02 269.24)
 		(diameter 0)
@@
 	)
 	(junction
-		(at 224.79 259.08)
-		(diameter 0)
-		(color 0 0 0 0)
-	)
-	(junction
 		(at 140.97 35.56)
 		(diameter 0)
@@
 	(wire
 		(pts
+			(xy 261.62 260.35) (xy 260.35 260.35)
+		)
+		(stroke
+			(width 0)
+			(type default)
+		)
+	)
+	(wire
+		(pts
 			(xy 41.91 199.39) (xy 45.72 199.39)
 		)
@@
 	(wire
 		(pts
-			(xy 236.22 266.7) (xy 236.22 269.24)
+			(xy 246.38 250.19) (xy 250.19 250.19)
+		)
+		(stroke
+			(width 0)
+			(type default)
+		)
+	)
+	(wire
+		(pts
+			(xy 236.22 265.43) (xy 236.22 269.24)
 		)
 		(stroke
@@
 	(wire
 		(pts
+			(xy 236.22 250.19) (xy 238.76 250.19)
+		)
+		(stroke
+			(width 0)
+			(type default)
+		)
+	)
+	(wire
+		(pts
 			(xy 160.02 266.7) (xy 160.02 269.24)
 		)
@@
 	(wire
 		(pts
+			(xy 236.22 250.19) (xy 236.22 252.73)
+		)
+		(stroke
+			(width 0)
+			(type default)
+		)
+	)
+	(wire
+		(pts
 			(xy 72.39 189.23) (xy 72.39 191.77)
 		)
@@
 	(wire
 		(pts
+			(xy 243.84 260.35) (xy 250.19 260.35)
+		)
+		(stroke
+			(width 0)
+			(type default)
+		)
+	)
+	(wire
+		(pts
 			(xy 69.85 259.08) (xy 86.36 259.08)
 		)
@@
 	(wire
 		(pts
-			(xy 210.82 259.08) (xy 214.63 259.08)
-		)
-		(stroke
-			(width 0)
-			(type default)
-		)
-	)
-	(wire
-		(pts
 			(xy 312.42 36.83) (xy 325.12 36.83)
 		)
@@
 	(wire
 		(pts
-			(xy 222.25 259.08) (xy 224.79 259.08)
-		)
-		(stroke
-			(width 0)
-			(type default)
-		)
-	)
-	(wire
-		(pts
 			(xy 354.33 49.53) (xy 354.33 48.26)
 		)
@@
 	(wire
 		(pts
-			(xy 236.22 250.19) (xy 233.68 250.19)
-		)
-		(stroke
-			(width 0)
-			(type default)
-		)
-	)
-	(wire
-		(pts
 			(xy 290.83 228.6) (xy 290.83 231.14)
 		)
@@
 	(wire
 		(pts
-			(xy 224.79 259.08) (xy 224.79 250.19)
-		)
-		(stroke
-			(width 0)
-			(type default)
-		)
-	)
-	(wire
-		(pts
 			(xy 347.98 36.83) (xy 354.33 36.83)
 		)
@@
 	(wire
 		(pts
-			(xy 224.79 250.19) (xy 226.06 250.19)
-		)
-		(stroke
-			(width 0)
-			(type default)
-		)
-	)
-	(wire
-		(pts
 			(xy 38.1 105.41) (xy 40.64 105.41)
 		)
@@
 	(wire
 		(pts
+			(xy 252.73 260.35) (xy 250.19 260.35)
+		)
+		(stroke
+			(width 0)
+			(type default)
+		)
+	)
+	(wire
+		(pts
 			(xy 36.83 91.44) (xy 39.37 91.44)
 		)
@@
 	(wire
 		(pts
-			(xy 140.97 88.9) (xy 143.51 88.9)
+			(xy 250.19 250.19) (xy 250.19 260.35)
 		)
 		(stroke
@@
 	(wire
 		(pts
-			(xy 236.22 254) (xy 236.22 250.19)
+			(xy 140.97 88.9) (xy 143.51 88.9)
 		)
 		(stroke
@@
 	(wire
 		(pts
-			(xy 228.6 259.08) (xy 224.79 259.08)
-		)
-		(stroke
-			(width 0)
-			(type default)
-		)
-	)
-	(wire
-		(pts
 			(xy 137.16 78.74) (xy 140.97 78.74)
 		)
@@
 		)
 	)
-	(label "+3.3V_T"
-		(at 210.82 259.08 180)
-		(effects
-			(font
-				(size 1.27 1.27)
-			)
-			(justify right bottom)
-		)
-	)
 	(label "POTI"
 		(at 114.3 55.88 180)
@@
 		)
 	)
+	(label "+3.3V_T"
+		(at 261.62 260.35 0)
+		(effects
+			(font
+				(size 1.27 1.27)
+			)
+			(justify left bottom)
+		)
+	)
 	(label "DOS_OUTA"
 		(at 69.85 256.54 0)
@@
 	(symbol
 		(lib_id "rodl:AO3415_C840839")
-		(at 236.22 259.08 0)
+		(at 236.22 260.35 180)
 		(unit 1)
 		(exclude_from_sim no)
@@
 		(fields_autoplaced yes)
 		(property "Reference" "Q2"
-			(at 241.3 259.7149 0)
+			(at 231.14 257.1749 0)
 			(effects
 				(font
@@
 		)
 		(property "Value" "AO3415_C840839"
-			(at 241.3 262.2549 0)
+			(at 231.14 259.7149 0)
 			(effects
 				(font
@@
 		)
 		(property "Footprint" "rodl:SOT-23-3_L2.9-W1.6-P1.90-LS2.8-BR"
-			(at 236.22 274.32 0)
+			(at 236.22 245.11 0)
 			(effects
 				(font
@@
 		)
 		(property "Datasheet" "https://lcsc.com/product-detail/MOSFET_MDD-Microdiode-Electronics-AO3415_C840839.html"
-			(at 236.22 276.86 0)
+			(at 236.22 242.57 0)
 			(effects
 				(font
@@
 		)
 		(property "Description" ""
-			(at 236.22 259.08 0)
+			(at 236.22 260.35 0)
 			(effects
 				(font
@@
 		)
 		(property "LCSC Part" "C840839"
-			(at 236.22 279.4 0)
+			(at 236.22 240.03 0)
 			(effects
 				(font
@@
 		)
 		(instances
-			(project ""
+			(project "rodl"
 				(path "/23e7b4c4-dd72-4182-80ee-a7cc0380e7f4"
 					(reference "Q2")
@@
 	(symbol
 		(lib_id "Device:R")
-		(at 229.87 250.19 90)
+		(at 242.57 250.19 270)
 		(unit 1)
 		(exclude_from_sim no)
@@
 		(fields_autoplaced yes)
 		(property "Reference" "R8"
-			(at 229.87 243.84 90)
+			(at 242.57 243.84 90)
 			(effects
 				(font
@@
 		)
 		(property "Value" "10k"
-			(at 229.87 246.38 90)
+			(at 242.57 246.38 90)
 			(effects
 				(font
@@
 		)
 		(property "Footprint" "Resistor_SMD:R_0603_1608Metric"
-			(at 229.87 251.968 90)
+			(at 242.57 248.412 90)
 			(effects
 				(font
@@
 		)
 		(property "Datasheet" "~"
-			(at 229.87 250.19 0)
+			(at 242.57 250.19 0)
 			(effects
 				(font
@@
 		)
 		(property "Description" "Resistor"
-			(at 229.87 250.19 0)
+			(at 242.57 250.19 0)
 			(effects
 				(font
@@
 	(symbol
 		(lib_id "Device:R")
-		(at 218.44 259.08 90)
+		(at 256.54 260.35 270)
 		(unit 1)
 		(exclude_from_sim no)
@@
 		(on_board yes)
 		(dnp no)
-		(fields_autoplaced yes)
 		(property "Reference" "R9"
-			(at 218.44 252.73 90)
+			(at 256.54 264.16 90)
 			(effects
 				(font
@@
 		)
 		(property "Value" "1k"
-			(at 218.44 255.27 90)
+			(at 256.54 266.7 90)
 			(effects
 				(font
@@
 		)
 		(property "Footprint" "Resistor_SMD:R_0603_1608Metric"
-			(at 218.44 260.858 90)
+			(at 256.54 258.572 90)
 			(effects
 				(font
@@
 		)
 		(property "Datasheet" "~"
-			(at 218.44 259.08 0)
+			(at 256.54 260.35 0)
 			(effects
 				(font
@@
 		)
 		(property "Description" "Resistor"
-			(at 218.44 259.08 0)
+			(at 256.54 260.35 0)
 			(effects
 				(font
